Commit message: minor fixes

File: tm_description/xacro/macro.handsolo.urdf.xacro (robot description, xacro)
@@ -71,5 +71,5 @@
       <geometry>
         <!-- Scale the mesh to make it larger (1.5x in X and Y, keep Z the same) -->
-        <mesh filename="package://amr_visualisation/meshes/LD250.obj" scale="1.25 1.25 1.25"/>
+        <mesh filename="package://amr_description/meshes/LD250.obj" scale="1.25 1.25 1.25"/>
       </geometry>
       <material name="grey">
@@ -81,5 +81,5 @@
       <geometry>
         <!-- Scale the collision mesh to match the visual -->
-        <mesh filename="package://amr_visualisation/meshes/LD250.obj" scale="1.25 1.25 1.25"/>
+        <mesh filename="package://amr_description/meshes/LD250.obj" scale="1.25 1.25 1.25"/>
       </geometry>
     </collision>

Commit message: added laserframe to macro.handsolo xacro file

File: tm_description/xacro/macro.handsolo.urdf.xacro (robot description, xacro)
@@ -107,4 +107,10 @@
     </xacro:cylinder_inertial_z>
   </link>
+  <link name="${prefix}laser_frame"/>
+  <joint name="${prefix}base_link_to_laser_frame" type="fixed">
+    <parent link="${prefix}amr_base"/>
+    <child link="${prefix}laser_frame"/>
+    <origin xyz="0.45 0 0.195"/>
+  </joint>
   <!-- Joint connecting AMR base to arm base (link_0) -->
   <!-- IMPORTANT: The z offset must be at least half the height of the AMR base plus some clearance -->

Commit message: minor fix

File: tm_description/xacro/macro.handsolo.urdf.xacro (robot description, xacro)
@@ -107,10 +107,4 @@
     </xacro:cylinder_inertial_z>
   </link>
-  <link name="${prefix}laser_frame"/>
-  <joint name="${prefix}base_link_to_laser_frame" type="fixed">
-    <parent link="${prefix}amr_base"/>
-    <child link="${prefix}laser_frame"/>
-    <origin xyz="0.45 0 0.195"/>
-  </joint>
   <!-- Joint connecting AMR base to arm base (link_0) -->
   <!-- IMPORTANT: The z offset must be at least half the height of the AMR base plus some clearance -->
